File: micro_control_wireless.kicad_pcb (KiCad board)
At the start: 4 copper layers, 12.5 x 29.4 mm, 21 parts, among them J2 USB_B_Micro, U1 CH592F, U2 ME6211C33M5, Y1 Crystal_GND24

Commit message: small fixes
Routing:
- net GND: track 110.8 -> 108.7 mm
- net Net-(D1-K): track 6.80 -> 7.62 mm
- net (no net): vias 10 -> 11
Changed lines of the file:
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@@
 		(capping no)
 		(filling no)
-		(zone_defaults)
 		(pcbplotparams
 			(layerselection 0x00000000_00000000_55555555_5755f5ff)
@@
 	)
 	(via blind
-		(at 103.75 75.8)
+		(at 102.995174 75.101072)
 		(size 0.5)
 		(drill 0.3)
@@
 	)
 	(via blind
-		(at 96.95 75.8)
+		(at 96.9 76)
 		(size 0.5)
 		(drill 0.3)
@@
 	)
 	(via blind
-		(at 102.15 75.8)
+		(at 101.8125 75.4)
+		(size 0.5)
+		(drill 0.3)
+		(layers "F.Cu" "In1.Cu")
+		(net "")
+	)
+	(via blind
+		(at 104.1 75.9)
 		(size 0.5)
 		(drill 0.3)
@@
 	)
 	(segment
-		(start 96.841468 74.61)
-		(end 96.675734 74.775734)
-		(width 0.2)
-		(layer "F.Cu")
-		(net "GND")
-	)
-	(segment
 		(start 103.169411 63.619411)
 		(end 103.1 63.55)
@@
 	)
 	(segment
-		(start 97.25 74.61)
-		(end 96.841468 74.61)
-		(width 0.2)
-		(layer "F.Cu")
-		(net "GND")
-	)
-	(segment
 		(start 101.939411 71.139411)
 		(end 102.35 71.55)
@@
 	)
 	(segment
-		(start 99.85 61.3)
-		(end 99.85 62.55)
+		(start 96.35 74.2)
+		(end 96.431468 74.2)
 		(width 0.2)
 		(layer "F.Cu")
@@
 	)
 	(segment
-		(start 102.439411 63.871178)
-		(end 102.778822 63.871178)
+		(start 96.431468 74.2)
+		(end 96.841468 74.61)
 		(width 0.2)
 		(layer "F.Cu")
@@
 	)
 	(segment
-		(start 99.55 61)
-		(end 99.85 61.3)
+		(start 102.439411 63.871178)
+		(end 102.778822 63.871178)
 		(width 0.2)
 		(layer "F.Cu")
@@
 	)
 	(segment
-		(start 99.85 62.55)
-		(end 100.1 62.8)
+		(start 99.85 61.3)
+		(end 99.55 61)
+		(width 0.2)
+		(layer "F.Cu")
+		(net "GND")
+	)
+	(segment
+		(start 96.841468 74.61)
+		(end 97.25 74.61)
 		(width 0.2)
 		(layer "F.Cu")
@@
 	)
 	(segment
-		(start 97.4625 55.875)
-		(end 98.565 55.875)
+		(start 99.55 61)
+		(end 98.85 61)
 		(width 0.2)
 		(layer "F.Cu")
@@
 	)
 	(segment
-		(start 98.85 61)
-		(end 99.55 61)
+		(start 97.4625 55.875)
+		(end 98.565 55.875)
 		(width 0.2)
 		(layer "F.Cu")
@@
 	)
 	(via blind
-		(at 96.675734 74.775734)
+		(at 96.35 74.2)
 		(size 0.5)
 		(drill 0.3)
-		(layers "F.Cu" "B.Cu")
+		(layers "F.Cu" "In1.Cu")
 		(net "GND")
 	)
@@
 	)
 	(via blind
-		(at 100.1 62.8)
+		(at 99.85 61.3)
 		(size 0.5)
 		(drill 0.3)
@@
 	)
 	(segment
-		(start 102.99 75.2)
-		(end 102.0125 75.2)
-		(width 0.6)
-		(layer "B.Cu")
-		(net "GND")
-	)
-	(segment
 		(start 104.314644 75.164644)
 		(end 104.279288 75.2)
@@
 	)
 	(segment
-		(start 102.99 75.2)
-		(end 102.99 75.86)
-		(width 0.6)
+		(start 101.8125 75.4)
+		(end 102.79 75.4)
+		(width 0.2)
 		(layer "B.Cu")
 		(net "GND")
 	)
 	(segment
-		(start 102.0125 75.2)
-		(end 101.8125 75.4)
+		(start 102.99 75.2)
+		(end 102.99 75.86)
 		(width 0.6)
 		(layer "B.Cu")
@@
 	)
 	(segment
-		(start 98.778822 71.55)
-		(end 102.35 71.55)
+		(start 102.79 75.4)
+		(end 102.99 75.2)
 		(width 0.2)
-		(layer "In1.Cu")
+		(layer "B.Cu")
 		(net "GND")
 	)
 	(segment
-		(start 99.725 60.675)
-		(end 100.35 61.3)
+		(start 98.778822 71.55)
+		(end 102.35 71.55)
 		(width 0.2)
 		(layer "In1.Cu")
@@
 	)
 	(segment
-		(start 100.35 61.3)
-		(end 100.35 62.55)
-		(width 0.2)
-		(layer "In1.Cu")
-		(net "GND")
-	)
-	(segment
 		(start 97.07 73.8)
 		(end 96.35 73.8)
@@
 	)
 	(segment
-		(start 102.35 62.8)
-		(end 103.1 63.55)
+		(start 103.45 65.25)
+		(end 103.6 65.4)
 		(width 0.2)
 		(layer "In1.Cu")
@@
 	)
 	(segment
-		(start 103.45 65.25)
-		(end 103.6 65.4)
+		(start 96.871445 71.878555)
+		(end 97.15 71.6)
 		(width 0.2)
 		(layer "In1.Cu")
@@
 	)
 	(segment
-		(start 96.871445 71.878555)
-		(end 97.15 71.6)
+		(start 101.35 62.8)
+		(end 102.35 62.8)
 		(width 0.2)
 		(layer "In1.Cu")
@@
 	)
 	(segment
-		(start 100.1 62.8)
-		(end 102.35 62.8)
+		(start 102.35 62.8)
+		(end 103.1 63.55)
 		(width 0.2)
 		(layer "In1.Cu")
@@
 	)
 	(segment
+		(start 99.85 61.3)
+		(end 101.35 62.8)
+		(width 0.2)
+		(layer "In1.Cu")
+		(net "GND")
+	)
+	(segment
 		(start 96.35 74.45)
 		(end 97.1 75.2)
@@
 	)
 	(segment
+		(start 99.85 61.3)
+		(end 99.85 60.8)
+		(width 0.2)
+		(layer "In1.Cu")
+		(net "GND")
+	)
+	(segment
 		(start 97.6 73.27)
 		(end 97.07 73.8)
@@
 	)
 	(segment
-		(start 100.35 62.55)
-		(end 100.1 62.8)
-		(width 0.2)
-		(layer "In1.Cu")
-		(net "GND")
-	)
-	(segment
 		(start 104.687144 74.837144)
 		(end 105.05 75.2)
@@
 	)
 	(segment
+		(start 99.85 60.8)
+		(end 99.725 60.675)
+		(width 0.2)
+		(layer "In1.Cu")
+		(net "GND")
+	)
+	(segment
 		(start 97.39631 72.916311)
 		(end 97.6 73.120001)
@@
 	)
 	(segment
+		(start 101.775 63.375)
+		(end 101.4 63.75)
+		(width 0.2)
+		(layer "F.Cu")
+		(net "3.3V")
+	)
+	(segment
 		(start 104.1 60.01)
 		(end 104.31 60.01)
@@
 	)
 	(segment
-		(start 101.4 63.75)
-		(end 101.4 64.35)
-		(width 0.2)
-		(layer "F.Cu")
-		(net "3.3V")
-	)
-	(segment
 		(start 101.251471 65.648529)
 		(end 101.534314 65.931371)
@@
 	)
 	(segment
-		(start 104.1 61.05)
-		(end 104.35 61.05)
+		(start 101.4 63.75)
+		(end 101.4 64.35)
 		(width 0.2)
 		(layer "F.Cu")
@@
 	)
 	(segment
-		(start 101.6 64.55)
-		(end 101.760589 64.55)
+		(start 101.4 64.35)
+		(end 101.6 64.55)
+		(width 0.2)
+		(layer "F.Cu")
+		(net "3.3V")
+	)
+	(segment
+		(start 104.1 61.05)
+		(end 104.35 61.05)
 		(width 0.2)
 		(layer "F.Cu")
@@
 	)
 	(segment
+		(start 101.6 64.55)
+		(end 101.760589 64.55)
+		(width 0.2)
+		(layer "F.Cu")
+		(net "3.3V")
+	)
+	(segment
 		(start 102.125 61.05)
 		(end 102.85 61.05)
@@
 	)
 	(segment
-		(start 101.4 64.35)
-		(end 101.6 64.55)
-		(width 0.2)
-		(layer "F.Cu")
-		(net "3.3V")
-	)
-	(segment
 		(start 104.1 60.01)
 		(end 104.1 60.4)
@@
 	)
 	(via blind
-		(at 101.4 63.75)
+		(at 101.775 63.375)
 		(size 0.5)
 		(drill 0.3)
@@
 	)
 	(segment
+		(start 101.775 63.375)
+		(end 102.475 62.675)
+		(width 0.2)
+		(layer "In2.Cu")
+		(net "3.3V")
+	)
+	(segment
 		(start 104.85 60.55)
 		(end 104.85 64.05)
@@
 	)
 	(segment
-		(start 101.4 63.75)
-		(end 102.475 62.675)
-		(width 0.2)
-		(layer "In2.Cu")
-		(net "3.3V")
-	)
-	(segment
 		(start 104.85 64.05)
 		(end 103.725 65.175)
@@
 	)
 	(segment
-		(start 95.8125 63.8375)
-		(end 95.35 63.8375)
+		(start 95.325589 60.78)
+		(end 95.325589 62.238089)
+		(width 0.2)
+		(layer "F.Cu")
+		(net "Net-(D1-A)")
+	)
+	(segment
+		(start 95.325589 62.238089)
+		(end 95.35 62.2625)
+		(width 0.2)
+		(layer "F.Cu")
+		(net "Net-(D1-A)")
+	)
+	(segment
+		(start 97.8 62.7)
+		(end 96.4875 62.7)
 		(width 0.2)
 		(layer "F.Cu")
@@
 	)
 	(segment
-		(start 100.402943 64.8)
-		(end 100.402943 64.102943)
+		(start 98.3 63.2)
+		(end 97.8 62.7)
 		(width 0.2)
 		(layer "F.Cu")
@@
 	)
 	(segment
-		(start 99 62.7)
-		(end 96.95 62.7)
+		(start 100.9 64.3)
+		(end 100.9 63.9)
 		(width 0.2)
 		(layer "F.Cu")
@@
 	)
 	(segment
-		(start 96.95 62.7)
-		(end 95.8125 63.8375)
+		(start 100.9 63.9)
+		(end 100.2 63.2)
 		(width 0.2)
 		(layer "F.Cu")
@@
 	)
 	(segment
-		(start 100.402943 64.102943)
-		(end 99 62.7)
+		(start 96.4875 62.7)
+		(end 95.35 63.8375)
 		(width 0.2)
 		(layer "F.Cu")
@@
 	)
 	(segment
-		(start 95.325589 60.78)
-		(end 95.325589 62.238089)
+		(start 100.2 63.2)
+		(end 98.3 63.2)
 		(width 0.2)
 		(layer "F.Cu")
-		(net "Net-(D1-A)")
+		(net "Net-(D1-K)")
 	)
 	(segment
-		(start 95.325589 62.238089)
-		(end 95.35 62.2625)
+		(start 100.402943 64.797057)
+		(end 100.9 64.3)
 		(width 0.2)
 		(layer "F.Cu")
-		(net "Net-(D1-A)")
+		(net "Net-(D1-K)")
+	)
+	(segment
+		(start 100.402943 64.8)
+		(end 100.402943 64.797057)
+		(width 0.2)
+		(layer "F.Cu")
+		(net "Net-(D1-K)")
 	)
 	(segment
